File: AWS_CPU_Motherboard/AWS_CPU_Motherboard.kicad_pcb (KiCad board)
At the start: 4 copper layers, 255 x 305 mm, 53 parts, among them J1 Power, J10 UART B, J12 Video, J14 HDD Power, J15 HDD Power, J2 Speaker, J3 Cluster, J4 Cluster, J5 HDD Power, J6 Drive Type, J7 Keyboard, J8 Printer Interface, J9 UART A, Q2 Q_NPN_CBE, SW1 Reset, U1 CPU, U2 Floppy 0, U3 Floppy 1, U4 MFM/Floppy, U5 MFM Control, U6 MFM Data, U7 AM26LV32xD, U8 74LS86

Commit message: Clean up old code
Parts:
- added REF**: CPU_Board, AWS:CPU_Board, F.Cu at (580.9, 284.4)
- moved REF** 425.0 mm to (1005.8, 289.8)
Connections:
- U4 pad 6: 2SIDED- -> unconnected-(U4-2SIDED--Pad6)
Routing:
- net 2SIDED-: track 180.9 -> 171.6 mm, vias 1 -> 2
Other:
- outline, holes or cut-outs redrawn
