File: AWS_CPU_Motherboard/AWS_CPU_Motherboard.kicad_sch (KiCad schematic)
At the start: 52 parts, among them J1 Power, J10 UART B, J12 Video, J14 HDD Power, J15 HDD Power, J2 Speaker, J3 Cluster, J4 Cluster, J5 HDD Power, J6 Drive Type, J7 Keyboard, J8 Printer Interface, J9 UART A, Q2 Q_NPN_CBE, SW1 Reset, U1 CPU, U2 Floppy 0, U3 Floppy 1, U4 MFM/Floppy, U5 MFM Control, U6 MFM Data, U7 AM26LV32xD, U8 74LS86

Commit message: Clean up old code
Connections:
- net 2SIDED-: no longer U4.6 (2SIDED-)
- no-connect marks 41 -> 42
Other:
- note added: "Note that Pin 16 and Pin 17 are wired together on the hard drive controller. Pin 6 look to be unused. For the floppy to work pin 16/17 must go to flopy pin34"
Changed lines of the file:
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@@
 		)
 	)
+	(text "Note that Pin 16 and Pin 17 are wired together on the hard drive controller.\nPin 6 look to be unused.\n\nFor the floppy to work pin 16/17 must go to flopy pin34"
+		(exclude_from_sim no)
+		(at 315.722 141.478 0)
+		(effects
+			(font
+				(size 1.27 1.27)
+			)
+		)
+	)
 	(text "P10"
 		(exclude_from_sim no)
@@
 	)
 	(no_connect
+		(at 331.47 36.83)
+	)
+	(no_connect
 		(at 34.29 224.79)
 	)
@@
 	(wire
 		(pts
-			(xy 331.47 49.53) (xy 349.25 49.53)
-		)
-		(stroke
-			(width 0)
-			(type default)
-		)
-	)
-	(wire
-		(pts
 			(xy 422.91 120.65) (xy 427.99 120.65)
 		)
@@
 	(wire
 		(pts
-			(xy 349.25 36.83) (xy 349.25 49.53)
-		)
-		(stroke
-			(width 0)
-			(type default)
-		)
-	)
-	(wire
-		(pts
 			(xy 501.65 46.99) (xy 505.46 46.99)
 		)
@@
 	(wire
 		(pts
-			(xy 331.47 36.83) (xy 349.25 36.83)
-		)
-		(stroke
-			(width 0)
-			(type default)
-		)
-	)
-	(wire
-		(pts
 			(xy 78.74 340.36) (xy 99.06 340.36)
 		)
@@
 	(global_label "2SIDED-"
 		(shape input)
-		(at 349.25 49.53 0)
+		(at 331.47 49.53 0)
 		(fields_autoplaced yes)
 		(effects
@@
 		)
 		(property "Intersheetrefs" "${INTERSHEET_REFS}"
-			(at 360.5204 49.53 0)
+			(at 342.7404 49.53 0)
 			(effects
 				(font
