File: AWS_CPU_Video_Decoder/AWS_CPU_Video_Decoder/AWS_CPU_Video_Decoder.kicad_sch (KiCad schematic)
At the start: 58 parts, among them J1 Conn_02x20_Odd_Even, J10 Conn_01x04_Pin, J11 Conn_01x04_Pin, J12 Conn_01x04_Pin, J13 Conn_01x04_Pin, J14 Conn_01x04_Pin, J15 Conn_01x04_Pin, J16 Video, J18 Conn_01x02_Pin, J19 Conn_01x02_Pin, J2 Conn_01x04_Pin, J3 Video, J4 Conn_01x04_Pin, J5 Conn_02x20_Odd_Even, J6 Conn_01x04_Pin, J7 Conn_01x04_Pin, J8 Conn_01x04_Pin, J9 Conn_01x04_Pin, SW1 Reset

Commit message: Clean up old code
Other:
- note removed: "Note: use 19,20,21 for video"
Changed lines of the file:
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@@
-		)
-	)
-	(text "Note: use 19,20,21 for video"
-		(exclude_from_sim no)
-		(at 427.99 70.866 0)
-		(effects
-			(font
-				(size 1.27 1.27)
-			)
 		)
 	)

Commit message: Added rotary encoder for switching mode and scrolling
Parts:
- added J20: Encoder, Connector_PinHeader_2.54mm:PinHeader_1x05_P2.54mm_Horizontal, symbol Connector_Generic:Conn_01x05
Connections:
- net +3V3: now also J20.5 (Pin_5)
- net GND: now also J20.1 (Pin_1)
- net GPIO26: now also J20.4 (Pin_4)
- net GPIO27: now also J20.3 (Pin_3)
- net GPIO28: now also J20.2 (Pin_2)
Other:
- note added: "AWS Pinout"
- note added: "Level Shifters"
- note added: "MCU"
- note added: "Rotary Encoder"
- note added: "Video"
- moved on the sheet: A2, D1, H1, J1, J10, J11, J12, J13, J14, J15, J18, J19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
